File: Com_Comp.kicad_sch (KiCad schematic)
At the start: 10 parts, among them IC1 SX1278IMLTRT, U2 STM32L552CCU6, U2 Teseo-LIV3FL

Commit message: changed rf module to ZETA-433-SO
Parts:
- removed IC1: SX1278IMLTRT, QFN65P600X600X100-29N-D, symbol SX1278IMLTRT:SX1278IMLTRT
- added U5: ZETA-433-SO, symbol RF_AM_FM:ZETA-433-SO
Changed lines of the file:
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@@
-    )
-  )
-  (symbol (lib_id "SX1278IMLTRT:SX1278IMLTRT") (at 247.65 107.95 180) (unit 1)
-    (in_bom yes) (on_board yes) (dnp no) (fields_autoplaced)
-    (property "Reference" "IC1" (at 251.46 87.2139 0)
-      (effects (font (size 1.27 1.27)))
-    )
-    (property "Value" "SX1278IMLTRT" (at 251.46 89.7539 0)
-      (effects (font (size 1.27 1.27)))
-    )
-    (property "Footprint" "QFN65P600X600X100-29N-D" (at 210.82 25.73 0)
-      (effects (font (size 1.27 1.27)) (justify left top) hide)
-    )
-    (property "Datasheet" "https://datasheet.datasheetarchive.com/originals/distributors/DKDS-37/728736.pdf" (at 210.82 -74.27 0)
-      (effects (font (size 1.27 1.27)) (justify left top) hide)
-    )
-    (property "Height" "1" (at 210.82 -274.27 0)
-      (effects (font (size 1.27 1.27)) (justify left top) hide)
-    )
-    (property "Manufacturer_Name" "SEMTECH" (at 210.82 -374.27 0)
-      (effects (font (size 1.27 1.27)) (justify left top) hide)
-    )
-    (property "Manufacturer_Part_Number" "SX1278IMLTRT" (at 210.82 -474.27 0)
-      (effects (font (size 1.27 1.27)) (justify left top) hide)
-    )
-    (property "Mouser Part Number" "947-SX1278IMLTRT" (at 210.82 -574.27 0)
-      (effects (font (size 1.27 1.27)) (justify left top) hide)
-    )
-    (property "Mouser Price/Stock" "https://www.mouser.co.uk/ProductDetail/Semtech/SX1278IMLTRT?qs=rBWM4%252BvDhIee37k32BFwWg%3D%3D" (at 210.82 -674.27 0)
-      (effects (font (size 1.27 1.27)) (justify left top) hide)
-    )
-    (property "Arrow Part Number" "SX1278IMLTRT" (at 210.82 -774.27 0)
-      (effects (font (size 1.27 1.27)) (justify left top) hide)
-    )
-    (property "Arrow Price/Stock" "https://www.arrow.com/en/products/sx1278imltrt/semtech?region=nac" (at 210.82 -874.27 0)
-      (effects (font (size 1.27 1.27)) (justify left top) hide)
-    )
-    (pin "1")
-    (pin "10")
-    (pin "11")
-    (pin "12")
-    (pin "13")
-    (pin "14")
-    (pin "15")
-    (pin "16")
-    (pin "17")
-    (pin "18")
-    (pin "19")
-    (pin "2")
-    (pin "20")
-    (pin "21")
-    (pin "22")
-    (pin "23")
-    (pin "24")
-    (pin "25")
-    (pin "26")
-    (pin "27")
-    (pin "28")
-    (pin "29")
-    (pin "3")
-    (pin "4")
-    (pin "5")
-    (pin "6")
-    (pin "7")
-    (pin "8")
-    (pin "9")
-    (instances
-      (project "Flight-Computer"
-        (path "/3ff93668-efc3-42e6-a72e-521229bcc4c8/34cd6572-1d03-4ef0-8710-332eddd1e16e"
-          (reference "IC1") (unit 1)
-        )
-      )
     )
   )
@@
         )
       )
+    )
+  )
+  (symbol (lib_id "RF_AM_FM:ZETA-433-SO") (at 220.98 99.06 180) (unit 1)
+    (in_bom yes) (on_board yes) (dnp no) (fields_autoplaced)
+    (property "Reference" "U5" (at 221.3259 83.82 0)
+      (effects (font (size 1.27 1.27)) (justify right))
+    )
+    (property "Value" "ZETA-433-SO" (at 221.3259 86.36 0)
+      (effects (font (size 1.27 1.27)) (justify right))
+    )
+    (property "Footprint" "" (at 229.87 105.41 0)
+      (effects (font (size 1.27 1.27)) hide)
+    )
+    (property "Datasheet" "https://www.rfsolutions.co.uk/downloads/1456219226DS-ZETA.pdf" (at 227.33 107.95 0)
+      (effects (font (size 1.27 1.27)) hide)
+    )
+    (pin "7")
+    (pin "8")
+    (pin "6")
+    (pin "12")
+    (pin "2")
+    (pin "11")
+    (pin "3")
+    (pin "9")
+    (pin "1")
+    (pin "5")
+    (pin "4")
+    (pin "10")
+    (instances
+      (project "Flight-Computer"
+        (path "/3ff93668-efc3-42e6-a72e-521229bcc4c8/34cd6572-1d03-4ef0-8710-332eddd1e16e"
+          (reference "U5") (unit 1)
+        )
+      )
