File: Flight-Computer.kicad_sch (KiCad schematic)
At the start: 5 parts, among them U1 STM32U575RIT6, U2 STM32L552CCU6, U3 BNO055, U4 MS5611-01BA

Commit message: Arbeit von Makerspace
Parts:
- added U5: STM32L552CCUx, Package_DFN_QFN:QFN-48-1EP_7x7mm_P0.5mm_EP5.6x5.6mm, symbol MCU_ST_STM32L5:STM32L552CCUx
Connections:
- new net: U5.23 (VSS), U5.35 (VSS), U5.47 (VSS), U5.49 (VSS)
Other:
- moved on the sheet: AC1, U2, U3, U4

Commit message: Added RF chips and Pages in Sch.
Parts:
- removed AC1: H3LIS331DLTR, LIS3DHTR, symbol H3LIS331DLTR:H3LIS331DLTR
- removed U2: STM32L552CCU6, Package_DFN_QFN:QFN-48-1EP_7x7mm_P0.5mm_EP5.6x5.6mm, symbol MCU_ST_STM32L5:STM32L552CCUx
- removed U3: BNO055, Package_LGA:LGA-28_5.2x3.8mm_P0.5mm, symbol Sensor_Motion:BNO055
- removed U4: MS5611-01BA, Package_LGA:LGA-8_3x5mm_P1.25mm, symbol Sensor_Pressure:MS5611-01BA
- removed U5: STM32L552CCUx, Package_DFN_QFN:QFN-48-1EP_7x7mm_P0.5mm_EP5.6x5.6mm, symbol MCU_ST_STM32L5:STM32L552CCUx
- added C1, C17, C2, C3, C4, C5: 100n, symbol Device:C
- added C18, C6, C7: 10u, symbol Device:C
Connections:
- net +3.3V: now also C1.1, C2.1, C3.1, C4.1, C5.1, C6.1, C7.1
- net GND: now also C1.2, C17.2, C18.2, C2.2, C3.2, C4.2, C5.2, C6.2, C7.2
- net +3.3VA: now reaches U1.13 (VDDA)
- net +3.3VA: now also C17.1, C18.1
Other:
- added sheet BMS+PSU (BMS+PSU.kicad_sch)
- added sheet Comms Computer (Com_Comp.kicad_sch)
- added sheet Measurement Computer (Mes_Comp.kicad_sch)
- moved on the sheet: U1

Commit message: changed rf module to ZETA-433-SO
Parts:
- added U4: MT25QUxxxxxx1xW7, Package_DFN_QFN:W-PDFN-8-1EP_6x5mm_P1.27mm_EP3x3mm, symbol Memory_Flash:MT25QUxxxxxx1xW7
Changed lines of the file:
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@@
+    )
+  )
+  (symbol (lib_id "Memory_Flash:MT25QUxxxxxx1xW7") (at 184.15 99.06 0) (unit 1)
+    (in_bom yes) (on_board yes) (dnp no) (fields_autoplaced)
+    (property "Reference" "U4" (at 193.04 97.79 0)
+      (effects (font (size 1.27 1.27)) (justify left))
+    )
+    (property "Value" "MT25QUxxxxxx1xW7" (at 193.04 100.33 0)
+      (effects (font (size 1.27 1.27)) (justify left))
+    )
+    (property "Footprint" "Package_DFN_QFN:W-PDFN-8-1EP_6x5mm_P1.27mm_EP3x3mm" (at 204.47 96.52 0)
+      (effects (font (size 1.27 1.27)) hide)
+    )
+    (property "Datasheet" "https://media-www.micron.com/-/media/client/global/documents/products/data-sheet/nor-flash/serial-nor/mt25q/die-rev-a/mt25q_qljs_u_256_aba_0.pdf" (at 184.15 81.28 0)
+      (effects (font (size 1.27 1.27)) hide)
+    )
+    (pin "1")
+    (pin "2")
+    (pin "3")
+    (pin "4")
+    (pin "5")
+    (pin "6")
+    (pin "7")
+    (pin "8")
+    (pin "9")
+    (instances
+      (project "Flight-Computer"
+        (path "/3ff93668-efc3-42e6-a72e-521229bcc4c8"
+          (reference "U4") (unit 1)
+        )
+      )
     )
   )
